File: LoRaESP32.kicad_pcb (KiCad board)
At the start: 2 copper layers, 81 x 62 mm, 61 parts, among them J1 TYPE-C 16PIN 2MD(073), SW3 EC11E1834403, U2 TPS63001, U3 ESP32-S3-WROOM-1, U4 MCP73871-2CC, U5 Ra-01SH

Commit message: Add files via upload
Routing:
- net Row4: track 56.2 -> 75.7 mm
- net Row3: track 43.2 -> 62.7 mm
- net Row2: track 35.7 -> 55.2 mm
- net Row1: track 28.2 -> 47.7 mm
Changed lines of the file:
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@@
+	)
+	(segment
+		(start 23.05 49.65)
+		(end 29.55 49.65)
+		(width 0.3)
+		(layer "B.Cu")
+		(net 32)
+	)
+	(segment
+		(start 32.8 49.65)
+		(end 39.3 49.65)
+		(width 0.5)
+		(layer "B.Cu")
+		(net 32)
+	)
+	(segment
+		(start 42.45 49.65)
+		(end 48.95 49.65)
+		(width 0.5)
+		(layer "B.Cu")
+		(net 32)
 	)
 	(segment
@@
 		(width 0.5)
 		(layer "F.Cu")
+		(net 35)
+	)
+	(segment
+		(start 23.05 67.3)
+		(end 29.55 67.3)
+		(width 0.3)
+		(layer "B.Cu")
+		(net 35)
+	)
+	(segment
+		(start 42.45 67.3)
+		(end 48.95 67.3)
+		(width 0.5)
+		(layer "B.Cu")
+		(net 35)
+	)
+	(segment
+		(start 32.85 67.3)
+		(end 39.35 67.3)
+		(width 0.5)
+		(layer "B.Cu")
 		(net 35)
 	)
@@
 		(width 0.5)
 		(layer "F.Cu")
+		(net 47)
+	)
+	(segment
+		(start 29.55 58.55)
+		(end 23.05 58.55)
+		(width 0.5)
+		(layer "B.Cu")
+		(net 47)
+	)
+	(segment
+		(start 48.95 58.55)
+		(end 42.45 58.55)
+		(width 0.5)
+		(layer "B.Cu")
+		(net 47)
+	)
+	(segment
+		(start 39.35 58.55)
+		(end 32.85 58.55)
+		(width 0.5)
+		(layer "B.Cu")
 		(net 47)
 	)
@@
 	)
 	(segment
+		(start 22.95 75.55)
+		(end 29.45 75.55)
+		(width 0.3)
+		(layer "B.Cu")
+		(net 62)
+	)
+	(segment
 		(start 73.85 46.31005)
 		(end 73.85 41.9)
 		(width 0.5)
 		(layer "B.Cu")
+		(net 62)
+	)
+	(segment
+		(start 39.35 75.55)
+		(end 32.85 75.55)
+		(width 0.5)
+		(layer "B.Cu")
+		(net 62)
+	)
+	(segment
+		(start 48.95 75.55)
+		(end 42.45 75.55)
+		(width 0.5)
+		(layer "B.Cu")
